Commit message: Core Bot Edited

File: description/robot_core.xacro (robot description, xacro)
@@ -1,192 +1,54 @@
 <?xml version="1.0"?>
 <robot xmlns:xacro="http://www.ros.org/wiki/xacro" name="robot">
-    <material name="white">
-        <color rgba="1 1 1 1"/>
-    </material>
-    <material name="red">
-        <color rgba="1 0 0 1"/>
-    </material>
-    <material name="orange">
-        <color rgba="1 0.3 0.1 1"/>
-    </material>
-    <material name="blue">
-        <color rgba="0.2 0.2 1 1"/>
-    </material>
-    <material name="black">
-        <color rgba="0 0 0 1"/>
-    </material>
-    <material name="grey">
-         <color rgba="0.5 0.5 0.5 1"/>
-    </material>
-    <material name="wood">
-         <color rgba="0.5 0.3 0.1 1"/>
-    </material>
-    <!-- Box dimensions -->
-    <xacro:property name="box_length" value="0.394" />
-    <xacro:property name="box_width" value="0.300" />
-    <xacro:property name="box_height" value="0.280" />
-    <xacro:property name="wall_thickness" value="0.012" />
-    <xacro:property name="wall_mass" value="1.5" />
-    <!-- Additional mass properties -->
-    <xacro:property name="base_mass" value="2.0" />
-    <xacro:property name="motor_mass" value="1.5" />
-    <xacro:property name="wheel_mass" value="0.5" />
-    <xacro:property name="caster_mass" value="0.2" />
-    <!-- World link (fixed reference) -->
-    <link name="world"/>
-    <!-- Base joint connecting to world -->
-    <joint name="base_joint" type="fixed">
-        <origin xyz="0 0 0.063" rpy="0 0 0"/>
-        <parent link="world"/>
-        <child link="base_link"/>
+    <!-- ================= MATERIALS ================= -->
+    <material name="white"><color rgba="1 1 1 1"/></material>
+    <material name="black"><color rgba="0 0 0 1"/></material>
+    <material name="grey"><color rgba="0.5 0.5 0.5 1"/></material>
+    <!-- ================= PROPERTIES ================= -->
+    <xacro:property name="box_length" value="0.394"/>
+    <xacro:property name="box_width"  value="0.300"/>
+    <xacro:property name="box_height" value="0.280"/>
+    <!-- ================= BASE LINK ================= -->
+    <link name="base_link">
+        <inertial>
+            <origin xyz="0 0 0"/>
+            <mass value="0.5"/>
+            <inertia ixx="0.002" iyy="0.002" izz="0.002"
+                     ixy="0" ixz="0" iyz="0"/>
+        </inertial>
+    </link>
+    <!-- ================= CHASSIS ================= -->
+    <joint name="chassis_joint" type="fixed">
+        <origin xyz="-0.115 0 0"/>
+        <parent link="base_link"/>
+        <child link="chassis_link"/>
     </joint>
-    <!-- Base Link (reference frame at ground level - base plate) -->
-    <link name="base_link">
+    <link name="chassis_link">
         <visual>
-            <origin xyz="0.118 0 0" rpy="0 0 0"/>
+            <origin xyz="${box_length/2} 0 ${box_height/2}"/>
             <geometry>
-                <box size="0.394 0.300 0.012"/>
+                <box size="${box_length} ${box_width} ${box_height}"/>
             </geometry>
-            <material name="wood"/>
+            <material name="white"/>
         </visual>
         <collision>
-            <origin xyz="0.118 0 0" rpy="0 0 0"/>
+            <origin xyz="${box_length/2} 0 ${box_height/2}"/>
             <geometry>
-                <box size="0.394 0.300 0.012"/>
+                <box size="${box_length} ${box_width} ${box_height}"/>
             </geometry>
         </collision>
         <inertial>
-            <origin xyz="0.118 0 0" rpy="0 0 0"/>
-            <mass value="${base_mass}" />
-            <inertia ixx="${(base_mass/12) * (0.012*0.012 + box_width*box_width)}"
-                     ixy="0.0" ixz="0.0"
-                     iyy="${(base_mass/12) * (box_length*box_length + 0.012*0.012)}"
-                     iyz="0.0"
-                     izz="${(base_mass/12) * (box_length*box_length + box_width*box_width)}" />
+            <origin xyz="${box_length/2} 0 ${box_height/2}"/>
+            <mass value="8.0"/>
+            <inertia
+                ixx="${(1/12.0)*8*(box_width*box_width + box_height*box_height)}"
+                iyy="${(1/12.0)*8*(box_length*box_length + box_height*box_height)}"
+                izz="${(1/12.0)*8*(box_length*box_length + box_width*box_width)}"
+                ixy="0" ixz="0" iyz="0"/>
         </inertial>
     </link>
-    <!-- LEFT WALL -->
-    <joint name="left_joint" type="fixed">
-        <origin xyz="0.118 ${-(box_width/2 - wall_thickness/2)} ${box_height/2}" rpy="0 0 0"/>
-        <parent link="base_link"/>
-        <child link="left_link"/>
-    </joint>
-    <link name="left_link">
-        <visual>
-            <origin xyz="0 0 0" rpy="0 0 0"/>
-            <geometry>
-                <box size="${box_length} ${wall_thickness} ${box_height}"/>
-            </geometry>
-            <material name="wood"/>
-        </visual>
-        <collision>
-            <origin xyz="0 0 0" rpy="0 0 0"/>
-            <geometry>
-                <box size="${box_length} ${wall_thickness} ${box_height}"/>
-            </geometry>
-        </collision>
-        <inertial>
-            <origin xyz="0 0 0" rpy="0 0 0"/>
-            <mass value="${wall_mass}" />
-            <inertia ixx="${(wall_mass/12) * (wall_thickness*wall_thickness + box_height*box_height)}"
-                     ixy="0.0" ixz="0.0"
-                     iyy="${(wall_mass/12) * (box_length*box_length + box_height*box_height)}"
-                     iyz="0.0"
-                     izz="${(wall_mass/12) * (box_length*box_length + wall_thickness*wall_thickness)}" />
-        </inertial>
-    </link>
-    <!-- RIGHT WALL -->
-    <joint name="right_joint" type="fixed">
-        <origin xyz="0.118 ${box_width/2 - wall_thickness/2} ${box_height/2}" rpy="0 0 0"/>
-        <parent link="base_link"/>
-        <child link="right_link"/>
-    </joint>
-    <link name="right_link">
-        <visual>
-            <origin xyz="0 0 0" rpy="0 0 0"/>
-            <geometry>
-                <box size="${box_length} ${wall_thickness} ${box_height}"/>
-            </geometry>
-            <material name="wood"/>
-        </visual>
-        <collision>
-            <origin xyz="0 0 0" rpy="0 0 0"/>
-            <geometry>
-                <box size="${box_length} ${wall_thickness} ${box_height}"/>
-            </geometry>
-        </collision>
-        <inertial>
-            <origin xyz="0 0 0" rpy="0 0 0"/>
-            <mass value="${wall_mass}" />
-            <inertia ixx="${(wall_mass/12) * (wall_thickness*wall_thickness + box_height*box_height)}"
-                     ixy="0.0" ixz="0.0"
-                     iyy="${(wall_mass/12) * (box_length*box_length + box_height*box_height)}"
-                     iyz="0.0"
-                     izz="${(wall_mass/12) * (box_length*box_length + wall_thickness*wall_thickness)}" />
-        </inertial>
-    </link>
-    <!-- FRONT WALL -->
-    <joint name="front_joint" type="fixed">
-        <origin xyz="${box_length/2 - wall_thickness/2 + 0.118} 0 ${box_height/2}" rpy="0 0 0"/>
-        <parent link="base_link"/>
-        <child link="front_link"/>
-    </joint>
-    <link name="front_link">
-        <visual>
-            <origin xyz="0 0 0" rpy="0 0 0"/>
-            <geometry>
-                <box size="${wall_thickness} ${box_width - 2*wall_thickness} ${box_height}"/>
-            </geometry>
-            <material name="wood"/>
-        </visual>
-        <collision>
-            <origin xyz="0 0 0" rpy="0 0 0"/>
-            <geometry>
-                <box size="${wall_thickness} ${box_width - 2*wall_thickness} ${box_height}"/>
-            </geometry>
-        </collision>
-        <inertial>
-            <origin xyz="0 0 0" rpy="0 0 0"/>
-            <mass value="${wall_mass}" />
-            <inertia ixx="${(wall_mass/12) * ((box_width - 2*wall_thickness)*(box_width - 2*wall_thickness) + box_height*box_height)}"
-                     ixy="0.0" ixz="0.0"
-                     iyy="${(wall_mass/12) * (wall_thickness*wall_thickness + box_height*box_height)}"
-                     iyz="0.0"
-                     izz="${(wall_mass/12) * (wall_thickness*wall_thickness + (box_width - 2*wall_thickness)*(box_width - 2*wall_thickness))}" />
-        </inertial>
-    </link>
-    <!-- BACK WALL -->
-    <joint name="back_joint" type="fixed">
-        <origin xyz="${-(box_length/2 - wall_thickness/2) + 0.118} 0 ${box_height/2}" rpy="0 0 0"/>
-        <parent link="base_link"/>
-        <child link="back_link"/>
-    </joint>
-    <link name="back_link">
-        <visual>
-            <origin xyz="0 0 0" rpy="0 0 0"/>
-            <geometry>
-                <box size="${wall_thickness} ${box_width - 2*wall_thickness} ${box_height}"/>
-            </geometry>
-            <material name="wood"/>
-        </visual>
-        <collision>
-            <origin xyz="0 0 0" rpy="0 0 0"/>
-            <geometry>
-                <box size="${wall_thickness} ${box_width - 2*wall_thickness} ${box_height}"/>
-            </geometry>
-        </collision>
-        <inertial>
-            <origin xyz="0 0 0" rpy="0 0 0"/>
-            <mass value="${wall_mass}" />
-            <inertia ixx="${(wall_mass/12) * ((box_width - 2*wall_thickness)*(box_width - 2*wall_thickness) + box_height*box_height)}"
-                     ixy="0.0" ixz="0.0"
-                     iyy="${(wall_mass/12) * (wall_thickness*wall_thickness + box_height*box_height)}"
-                     iyz="0.0"
-                     izz="${(wall_mass/12) * (wall_thickness*wall_thickness + (box_width - 2*wall_thickness)*(box_width - 2*wall_thickness))}" />
-        </inertial>
-    </link>
-    <!-- LEFT MOTOR -->
+    <!-- ================= LEFT MOTOR ================= -->
     <joint name="left_motor_joint" type="fixed">
-        <origin xyz="0 ${box_width/2 - wall_thickness/2 - 0.048} 0" rpy="0 0 0"/>
+        <origin xyz="0 0.102 0"/>
         <parent link="base_link"/>
         <child link="left_motor_link"/>
@@ -207,16 +69,14 @@
         </collision>
         <inertial>
-            <origin xyz="0 0.036 -0.023" rpy="${pi/2} 0 0"/>
-            <mass value="${motor_mass}" />
-            <inertia ixx="${(motor_mass/12) * (3*0.023*0.023 + 0.126*0.126)}"
-                     ixy="0.0" ixz="0.0"
-                     iyy="${(motor_mass/12) * (3*0.023*0.023 + 0.126*0.126)}"
-                     iyz="0.0"
-                     izz="${(motor_mass/2) * (0.023*0.023)}" />
+            <origin xyz="0 0.036 -0.023"/>
+            <mass value="0.6"/>
+            <inertia
+                ixx="0.0009" iyy="0.0004" izz="0.0009"
+                ixy="0" ixz="0" iyz="0"/>
         </inertial>
     </link>
-    <!-- LEFT Wheel -->
+    <!-- ================= LEFT WHEEL ================= -->
     <joint name="left_wheel_joint" type="continuous">
-        <origin xyz="0 ${(0.120 - 0.038)} -0.023" rpy="-${pi/2} 0 0"/>
+        <origin xyz="0 0.082 -0.023" rpy="-${pi/2} 0 0"/>
         <parent link="left_motor_link"/>
         <child link="left_wheel_link"/>
@@ -225,5 +85,4 @@
     <link name="left_wheel_link">
         <visual>
-            <origin xyz="0 0 0" rpy="0 0 0"/>
             <geometry>
                 <cylinder radius="0.04" length="0.035"/>
@@ -232,5 +91,4 @@
         </visual>
         <collision>
-            <origin xyz="0 0 0" rpy="0 0 0"/>
             <geometry>
                 <cylinder radius="0.04" length="0.035"/>
@@ -238,16 +96,13 @@
         </collision>
         <inertial>
-            <origin xyz="0 0 0" rpy="0 0 0"/>
-            <mass value="${wheel_mass}" />
-            <inertia ixx="${(wheel_mass/12) * (3*0.04*0.04 + 0.035*0.035)}"
-                     ixy="0.0" ixz="0.0"
-                     iyy="${(wheel_mass/12) * (3*0.04*0.04 + 0.035*0.035)}"
-                     iyz="0.0"
-                     izz="${(wheel_mass/2) * (0.04*0.04)}" />
+            <mass value="0.4"/>
+            <inertia
+                ixx="0.00016" iyy="0.00032" izz="0.00016"
+                ixy="0" ixz="0" iyz="0"/>
         </inertial>
     </link>
-    <!-- Right MOTOR -->
+    <!-- ================= RIGHT MOTOR ================= -->
     <joint name="right_motor_joint" type="fixed">
-        <origin xyz="0 -${box_width/2 - wall_thickness/2 - 0.048} 0" rpy="0 0 0"/>
+        <origin xyz="0 -0.102 0"/>
         <parent link="base_link"/>
         <child link="right_motor_link"/>
@@ -268,16 +123,14 @@
         </collision>
         <inertial>
-            <origin xyz="0 -0.036 -0.023" rpy="-${pi/2} 0 0"/>
-            <mass value="${motor_mass}" />
-            <inertia ixx="${(motor_mass/12) * (3*0.023*0.023 + 0.126*0.126)}"
-                     ixy="0.0" ixz="0.0"
-                     iyy="${(motor_mass/12) * (3*0.023*0.023 + 0.126*0.126)}"
-                     iyz="0.0"
-                     izz="${(motor_mass/2) * (0.023*0.023)}" />
+            <origin xyz="0 -0.036 -0.023"/>
+            <mass value="0.6"/>
+            <inertia
+                ixx="0.0009" iyy="0.0004" izz="0.0009"
+                ixy="0" ixz="0" iyz="0"/>
         </inertial>
     </link>
-    <!-- RIGHT Wheel -->
+    <!-- ================= RIGHT WHEEL ================= -->
     <joint name="right_wheel_joint" type="continuous">
-        <origin xyz="0 -${(0.120 - 0.038)} -0.023" rpy="${pi/2} 0 0"/>
+        <origin xyz="0 -0.082 -0.023" rpy="${pi/2} 0 0"/>
         <parent link="right_motor_link"/>
         <child link="right_wheel_link"/>
@@ -286,5 +139,4 @@
     <link name="right_wheel_link">
         <visual>
-            <origin xyz="0 0 0" rpy="0 0 0"/>
             <geometry>
                 <cylinder radius="0.04" length="0.035"/>
@@ -293,5 +145,4 @@
         </visual>
         <collision>
-            <origin xyz="0 0 0" rpy="0 0 0"/>
             <geometry>
                 <cylinder radius="0.04" length="0.035"/>
@@ -299,16 +150,13 @@
         </collision>
         <inertial>
-            <origin xyz="0 0 0" rpy="0 0 0"/>
-            <mass value="${wheel_mass}" />
-            <inertia ixx="${(wheel_mass/12) * (3*0.04*0.04 + 0.035*0.035)}"
-                     ixy="0.0" ixz="0.0"
-                     iyy="${(wheel_mass/12) * (3*0.04*0.04 + 0.035*0.035)}"
-                     iyz="0.0"
-                     izz="${(wheel_mass/2) * (0.04*0.04)}" />
+            <mass value="0.4"/>
+            <inertia
+                ixx="0.00016" iyy="0.00032" izz="0.00016"
+                ixy="0" ixz="0" iyz="0"/>
         </inertial>
     </link>
-    <!-- Caster Wheel -->
+    <!-- ================= CASTER ================= -->
     <joint name="caster_wheel_joint" type="fixed">
-        <origin xyz="0.269 0 -0.0315" rpy="0 0 0"/>
+        <origin xyz="0.250 0 -0.0315"/>
         <parent link="base_link"/>
         <child link="caster_wheel_link"/>
@@ -316,5 +164,4 @@
     <link name="caster_wheel_link">
         <visual>
-            <origin xyz="0 0 0" rpy="0 0 0"/>
             <geometry>
                 <sphere radius="0.0315"/>
@@ -323,5 +170,4 @@
         </visual>
         <collision>
-            <origin xyz="0 0 0" rpy="0 0 0"/>
             <geometry>
                 <sphere radius="0.0315"/>
@@ -329,11 +175,8 @@
         </collision>
         <inertial>
-            <origin xyz="0 0 0" rpy="0 0 0"/>
-            <mass value="${caster_mass}" />
-            <inertia ixx="${(2/5) * caster_mass * 0.0315 * 0.0315}"
-                     ixy="0.0" ixz="0.0"
-                     iyy="${(2/5) * caster_mass * 0.0315 * 0.0315}"
-                     iyz="0.0"
-                     izz="${(2/5) * caster_mass * 0.0315 * 0.0315}" />
+            <mass value="0.2"/>
+            <inertia
+                ixx="0.00008" iyy="0.00008" izz="0.00008"
+                ixy="0" ixz="0" iyz="0"/>
         </inertial>
     </link>

Commit message: Gazebo Simulated Right & fixed some core problems

File: description/robot_core.xacro (robot description, xacro)
@@ -48,4 +48,9 @@
         </inertial>
     </link>
+    <gazebo reference="chassis_link">
+        <material>Gazebo/White</material>
+        <mu1>1.0</mu1>
+        <mu2>1.0</mu2>
+    </gazebo>
     <!-- ================= LEFT MOTOR ================= -->
     <joint name="left_motor_joint" type="fixed">
@@ -76,4 +81,7 @@
         </inertial>
     </link>
+    <gazebo reference="left_motor_link">
+        <material>Gazebo/Grey</material>
+    </gazebo>
     <!-- ================= LEFT WHEEL ================= -->
     <joint name="left_wheel_joint" type="continuous">
@@ -82,4 +90,6 @@
         <child link="left_wheel_link"/>
         <axis xyz="0 0 1"/>
+        <limit effort="100" velocity="10.0"/>
+        <dynamics damping="0.1" friction="0.1"/>
     </joint>
     <link name="left_wheel_link">
@@ -102,4 +112,9 @@
         </inertial>
     </link>
+    <gazebo reference="left_wheel_link">
+        <material>Gazebo/Black</material>
+            <mu1>1.0</mu1>
+        <mu2>1.0</mu2>
+    </gazebo>
     <!-- ================= RIGHT MOTOR ================= -->
     <joint name="right_motor_joint" type="fixed">
@@ -130,10 +145,15 @@
         </inertial>
     </link>
+    <gazebo reference="right_motor_link">
+        <material>Gazebo/Grey</material>
+    </gazebo>
     <!-- ================= RIGHT WHEEL ================= -->
     <joint name="right_wheel_joint" type="continuous">
-        <origin xyz="0 -0.082 -0.023" rpy="${pi/2} 0 0"/>
+        <origin xyz="0 -0.082 -0.023" rpy="-${pi/2} 0 0"/>
         <parent link="right_motor_link"/>
         <child link="right_wheel_link"/>
         <axis xyz="0 0 1"/>
+        <limit effort="100" velocity="10.0"/>
+        <dynamics damping="0.1" friction="0.1"/>
     </joint>
     <link name="right_wheel_link">
@@ -156,4 +176,9 @@
         </inertial>
     </link>
+    <gazebo reference="right_wheel_link">
+        <material>Gazebo/Black</material>
+        <mu1>1.0</mu1>
+        <mu2>1.0</mu2>
+    </gazebo>
     <!-- ================= CASTER ================= -->
     <joint name="caster_wheel_joint" type="fixed">
@@ -181,3 +206,37 @@
         </inertial>
     </link>
+    <gazebo reference="caster_wheel_link">
+        <material>Gazebo/Black</material>
+        <mu1>0.000001</mu1>
+        <mu2>0.000001</mu2>
+    </gazebo>
+    <gazebo>
+  <plugin
+    filename="gz-sim-diff-drive-system"
+    name="gz::sim::systems::DiffDrive">
+    <!-- Joints -->
+    <left_joint>left_wheel_joint</left_joint>
+    <right_joint>right_wheel_joint</right_joint>
+    <!-- Geometry -->
+    <wheel_separation>0.164</wheel_separation>
+    <wheel_radius>0.04</wheel_radius>
+    <!-- Limits -->
+    <max_linear_acceleration>10.0</max_linear_acceleration>
+    <odom_publish_frequency>100.0</odom_publish_frequency>
+    <!-- Frames -->
+    <odom_frame>odom</odom_frame>
+    <base_frame>base_link</base_frame>
+    <!-- Topics -->
+    <topic>cmd_vel</topic>
+    <odom_topic>odom</odom_topic>
+    <publish_odom>true</publish_odom>
+    <publish_odom_tf>true</publish_odom_tf>
+    <publish_wheel_tf>true</publish_wheel_tf>
+  </plugin>
+    <plugin filename="gz-sim-joint-state-publisher-system" name="gz::sim::systems::JointStatePublisher">
+                        <topic>/model/my_bot/joint_states</topic>
+            <joint_name>right_wheel_joint</joint_name>
+            <joint_name>left_wheel_joint</joint_name>
+    </plugin>
+</gazebo>
 </robot>
