Commit message: Update obstacle map and configuration files (twist_mux, params)

File: description/camera.xacro (robot description, xacro)
@@ -1,4 +1,7 @@
 <?xml version="1.0"?>
 <robot xmlns:xacro="http://www.ros.org/wiki/xacro">
+    <gazebo reference="camera_joint">
+        <preserveFixedJoint>true</preserveFixedJoint>
+    </gazebo>
     <joint name="camera_joint" type="fixed">
         <parent link="chassis_link"/>
@@ -13,11 +16,25 @@
             <material name="red"/>
         </visual>
+        <inertial>
+            <origin xyz="0 0 0"/>
+            <mass value="0.01"/>
+            <inertia ixx="0.000001" ixy="0" ixz="0" iyy="0.000001" iyz="0" izz="0.000001"/>
+        </inertial>
     </link>
-        <joint name="camera_optical_joint" type="fixed">
+    <gazebo reference="camera_optical_joint">
+        <preserveFixedJoint>true</preserveFixedJoint>
+    </gazebo>
+    <joint name="camera_optical_joint" type="fixed">
         <origin xyz="0 0 0" rpy="${-pi/2} 0 ${-pi/2}" />
         <parent link="camera_link" />
         <child link="camera_link_optical" />
     </joint>
-    <link name="camera_link_optical"></link>
+    <link name="camera_link_optical">
+        <inertial>
+            <origin xyz="0 0 0"/>
+            <mass value="0.001"/>
+            <inertia ixx="0.0000001" ixy="0" ixz="0" iyy="0.0000001" iyz="0" izz="0.0000001"/>
+        </inertial>
+    </link>
         <gazebo reference="camera_link">
         <sensor name="camera" type="camera">

File: description/gazebo_control.xacro (robot description, xacro)
@@ -6,6 +6,6 @@
             <left_joint>left_wheel_joint</left_joint>
             <right_joint>right_wheel_joint</right_joint>
-            <wheel_separation>0.35</wheel_separation>
-            <wheel_radius>0.05</wheel_radius>
+            <wheel_separation>0.368</wheel_separation>
+            <wheel_radius>0.04</wheel_radius>
             <!-- Input -->
             <topic>cmd_vel</topic>

File: description/lidar.xacro (robot description, xacro)
@@ -1,4 +1,7 @@
 <?xml version="1.0"?>
 <robot xmlns:xacro="http://www.ros.org/wiki/xacro" >
+    <gazebo reference="laser_joint">
+        <preserveFixedJoint>true</preserveFixedJoint>
+    </gazebo>
     <joint name="laser_joint" type="fixed">
         <parent link="chassis_link"/>
@@ -42,5 +45,5 @@
                 </range>
             </lidar>
-            <topic>scan</topic>
+            <topic>/scan</topic>
             <gz_frame_id>laser_frame</gz_frame_id>
         </sensor>

File: description/robot_core.xacro (robot description, xacro)
@@ -19,4 +19,12 @@
         </inertial>
     </link>
+    <!-- ================= BASE FOOTPRINT ================= -->
+    <joint name="base_footprint_joint" type="fixed">
+        <parent link="base_link"/>
+        <child link="base_footprint"/>
+        <origin xyz="0 0 0" rpy="0 0 0"/>
+    </joint>
+    <link name="base_footprint">
+    </link>
     <!-- ================= CHASSIS ================= -->
     <joint name="chassis_joint" type="fixed">
